File: kicad/encoder-board/encoder-board.kicad_pcb (KiCad board)
At the start: 2 copper layers, 30 x 40 mm, 6 parts, among them J1 Conn_01x04_Pin, SW1 RotaryEncoder_Switch

Commit message: PCB trace finished
Other:
- board text added: "2026.05.29"
- board text added: "github.com/mar0x/midi_controller"
Changed lines of the file:
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@@
 		(layer "Edge.Cuts")
+	)
+	(gr_text "github.com/mar0x/midi_controller"
+		(at 156.97 114.18 0)
+		(layer "B.SilkS")
+		(effects
+			(font
+				(size 0.8 0.8)
+				(thickness 0.1)
+			)
+			(justify left bottom mirror)
+		)
+	)
+	(gr_text "2026.05.29"
+		(at 150.13 116.09 0)
+		(layer "B.SilkS")
+		(effects
+			(font
+				(size 1 1)
+				(thickness 0.2)
+				(bold yes)
+			)
+			(justify left bottom mirror)
+		)
 	)
 	(segment
