File: kicad/midi_pro_micro/midi_pro_micro.kicad_pcb (KiCad board)
At the start: 2 copper layers, 170 x 40 mm, 29 parts, among them J1 DIN-5_180degree, J2 DIN-5_180degree, J3 Conn_01x12, J5 Conn_01x05, J6 Conn_01x04, J7 Conn_01x02, U1 ProMicro, U2 AT25xxx, U3 6N138

Commit message: Start PCB trace
Parts:
- added D1: D, Diode_SMD:D_SOD-323_HandSoldering, F.Cu at (165.6, 98.5)
- moved R17 1.02 mm to (168.0, 110.0), turned to 0 degrees
Connections:
- J3 pad 4: RIGHT_LED -> LEFT_LED
- U1 pad 10: unconnected-(U1-7,E6-Pad10) -> OK_LED
- U1 pad 19: unconnected-(U1-F5,A2,20-Pad19) -> DOWN_LED
- U1 pad 5: LEFT_BTN -> LEFT_LED
- U1 pad 6: unconnected-(U1-3,D0,SCL-Pad6) -> LEFT_BTN
- U1 pad 8: unconnected-(U1-5,C6-Pad8) -> UP_LED
Routing:
- net OK_BTN: track 0.00 -> 91.3 mm, vias 0 -> 1
- net UP_BTN: track 0.00 -> 73.1 mm
- net UP_LED: track 0.00 -> 72.7 mm
- net LEFT_BTN: track 0.00 -> 69.2 mm
- net RIGHT_BTN: track 0.00 -> 64.0 mm
- net LEFT_LED: track 0.00 -> 60.0 mm
- net OK_LED: track 0.00 -> 58.1 mm
- net MISO: track 0.00 -> 58.0 mm
- net SCK: track 0.00 -> 53.4 mm
- net MOSI: track 0.00 -> 53.2 mm
- net TX: track 0.00 -> 38.3 mm
- net ENC_A: track 0.00 -> 37.5 mm
- net ENC_B: track 0.00 -> 37.4 mm
- net OLED_CS: track 0.00 -> 30.8 mm, vias 0 -> 1
- net Net-(D1-A): track 0.00 -> 14.3 mm
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- added copper zone on B.Cu, net GND
- added copper zone on F.Cu, net GND

Commit message: PCB trace finished
Parts:
- added G***: LOGO, lib:mvr-logo-16x10, B.Cu at (85.9, 108.7)
- added REF**: KiCad-Logo2_8mm_SilkScreen, Symbol:KiCad-Logo2_8mm_SilkScreen, B.Cu at (213.2, 109.1)
- moved R12 7.36 mm to (131.5, 110.4)
Connections:
- U1 pad 10: OK_LED -> DOWN_LED
- U1 pad 19: DOWN_LED -> OK_LED
- U1 pad 20: DOWN_BTN -> RIGHT_BTN
- U1 pad 21: unconnected-(U1-VCC-Pad21) -> +5V
- U1 pad 5: LEFT_LED -> UP_LED
- U1 pad 6: LEFT_BTN -> UP_BTN
- U1 pad 7: UP_BTN -> LEFT_LED
- U1 pad 8: UP_LED -> LEFT_BTN
- U1 pad 9: RIGHT_BTN -> DOWN_BTN
Routing:
- net +5V: track 2.81 -> 182.2 mm
- net DOWN_BTN: track 5.85 -> 65.8 mm
- net DOWN_LED: track 0.00 -> 59.9 mm
- net EEPROM_CS: track 0.00 -> 57.3 mm, vias 0 -> 1
- net RX: track 11.0 -> 39.7 mm, vias 0 -> 1
- net OK_BTN: track 91.3 -> 112.4 mm, vias 1 -> 0
- net RIGHT_BTN: track 64.0 -> 84.9 mm
- net OK_LED: track 58.1 -> 77.3 mm
- net UP_LED: track 72.7 -> 61.2 mm
- net LEFT_LED: track 60.0 -> 69.6 mm
- net UP_BTN: track 73.1 -> 68.4 mm
- net Net-(U2-~{WP}): track 0.00 -> 4.21 mm
- net LEFT_BTN: track 69.2 -> 72.5 mm
- net MOSI: track 53.2 -> 52.7 mm
- net GND: vias 0 -> 58
Other:
- board text added: "2026.05.29"
- board text added: "github.com/mar0x/midi_controller"
